Commit message: Mounted a camera sensor at the end of gripper for prototyping

File: ros2_ws/src/arctos_description/urdf/arctos_gazebo.xacro (robot description, xacro)
@@ -1,5 +1,5 @@
 <?xml version="1.0" ?>
 <robot xmlns:xacro="http://www.ros.org/wiki/xacro">
-<!-- Gazebo (gz sim) plugins for the arm: joint state feedback and position hold -->
+<!-- Gazebo (gz sim) plugins for the arm: sensor rendering, joint state feedback and position hold -->
 <xacro:macro name="arctos_joint_position_controller" params="joint max_velocity">
   <plugin filename="gz-sim-joint-position-controller-system" name="gz::sim::systems::JointPositionController">
@@ -12,4 +12,8 @@
 </xacro:macro>
 <gazebo>
+  <!-- Renders the camera sensors; the stock empty.sdf world does not load it -->
+  <plugin filename="gz-sim-sensors-system" name="gz::sim::systems::Sensors">
+    <render_engine>ogre2</render_engine>
+  </plugin>
   <plugin filename="gz-sim-joint-state-publisher-system" name="gz::sim::systems::JointStatePublisher">
     <topic>/joint_states</topic>

File: ros2_ws/src/arctos_description/urdf/arctos_scene.urdf.xacro (robot description, xacro)
@@ -6,4 +6,5 @@
 <xacro:include filename="$(find arctos_description)/urdf/table.urdf.xacro" />
 <xacro:include filename="$(find arctos_description)/urdf/apriltag.urdf.xacro" />
+<xacro:include filename="$(find arctos_description)/urdf/camera.urdf.xacro" />
 <!-- Arm base on the table surface. At the home pose the gripper points along -Y of base_link -->
 <xacro:property name="base_y_on_table" value="0.45"/>
@@ -24,3 +25,7 @@
   <origin xyz="0 ${gripper_tip_y - tag_distance} 0.001" rpy="0 0 0"/>
 </xacro:apriltag>
+<!-- Eye-in-hand camera on the +X side of the gripper body, looking along the jaws (-Y of Gripper_1) -->
+<xacro:camera name="camera" parent="Gripper_1">
+  <origin xyz="0.051 -0.03 0" rpy="0 0 ${-pi / 2}"/>
+</xacro:camera>
 </robot>
